File: hardware/mainboard/keypad_inputs.kicad_sch (KiCad schematic)
At the start: 49 parts, among them SW10 Keypad_Contact, SW11 Keypad_Contact, SW12 Keypad_Contact, SW13 Keypad_Contact, SW14 Keypad_Contact, SW15 Keypad_Contact, SW16 Keypad_Contact, SW17 Keypad_Contact, SW18 Keypad_Contact, SW19 Keypad_Contact, SW2 Keypad_Contact, SW20 Keypad_Contact, SW21 Keypad_Contact, SW22 Keypad_Contact, SW23 Keypad_Contact, SW24 Keypad_Contact, SW25 Keypad_Contact, SW26 Keypad_Contact, SW27 Keypad_Contact, SW28 Keypad_Contact, SW29 Keypad_Contact, SW3 Keypad_Contact, SW30 Keypad_Contact, SW31 Keypad_Contact, SW32 Keypad_Contact, SW33 Keypad_Contact, SW34 Keypad_Contact, SW35 Keypad_Contact, SW36 Keypad_Contact, SW37 Keypad_Contact, SW38 Keypad_Contact, SW39 Keypad_Contact, SW4 Keypad_Contact, SW40 Keypad_Contact, SW41 Keypad_Contact, SW42 Keypad_Contact, SW43 Keypad_Contact, SW44 Keypad_Contact, SW45 Keypad_Contact, SW46 Keypad_Contact, SW47 Keypad_Contact, SW48 Keypad_Contact, SW49 Keypad_Contact, SW5 Keypad_Contact, SW50 Keypad_Contact, SW6 Keypad_Contact, SW7 Keypad_Contact, SW8 Keypad_Contact, SW9 Keypad_Contact

Commit message: Refine keypad contacts and mechanical alignment
Parts:
- SW10, SW11, SW12, SW13, SW14, SW15, SW16, SW17, SW18, SW19, SW2, SW20, SW21, SW22, SW23, SW24, SW25, SW26, SW27, SW28, SW29, SW3, SW30, SW31, SW32, SW33, SW34, SW35, SW36, SW37, SW38, SW39, SW4, SW40, SW41, SW42, SW43, SW44, SW45, SW46, SW47, SW48, SW49, SW5, SW50, SW6, SW7, SW8, SW9: footprint CalcText:keypad_trace_button -> (none)
Changed lines of the file:
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@@
 			)
 		)
-		(property "Footprint" "CalcText:keypad_trace_button"
+		(property "Footprint" ""
 			(at 74.93 121.92 0)
 			(effects
@@
 			)
 		)
-		(property "Footprint" "CalcText:keypad_trace_button"
+		(property "Footprint" ""
 			(at 74.93 109.22 0)
 			(effects
@@
 			)
 		)
-		(property "Footprint" "CalcText:keypad_trace_button"
+		(property "Footprint" ""
 			(at 189.23 121.92 0)
 			(effects
@@
 			)
 		)
-		(property "Footprint" "CalcText:keypad_trace_button"
+		(property "Footprint" ""
 			(at 170.18 71.12 0)
 			(effects
@@
 			)
 		)
-		(property "Footprint" "CalcText:keypad_trace_button"
+		(property "Footprint" ""
 			(at 74.93 83.82 0)
 			(effects
@@
 			)
 		)
-		(property "Footprint" "CalcText:keypad_trace_button"
+		(property "Footprint" ""
 			(at 113.03 71.12 0)
 			(effects
@@
 			)
 		)
-		(property "Footprint" "CalcText:keypad_trace_button"
+		(property "Footprint" ""
 			(at 93.98 71.12 0)
 			(effects
@@
 			)
 		)
-		(property "Footprint" "CalcText:keypad_trace_button"
+		(property "Footprint" ""
 			(at 189.23 71.12 0)
 			(effects
@@
 			)
 		)
-		(property "Footprint" "CalcText:keypad_trace_button"
+		(property "Footprint" ""
 			(at 151.13 45.72 0)
 			(effects
@@
 			)
 		)
-		(property "Footprint" "CalcText:keypad_trace_button"
+		(property "Footprint" ""
 			(at 151.13 109.22 0)
 			(effects
@@
 			)
 		)
-		(property "Footprint" "CalcText:keypad_trace_button"
+		(property "Footprint" ""
 			(at 113.03 121.92 0)
 			(effects
@@
 			)
 		)
-		(property "Footprint" "CalcText:keypad_trace_button"
+		(property "Footprint" ""
 			(at 74.93 71.12 0)
 			(effects
@@
 			)
 		)
-		(property "Footprint" "CalcText:keypad_trace_button"
+		(property "Footprint" ""
 			(at 151.13 58.42 0)
 			(effects
@@
 			)
 		)
-		(property "Footprint" "CalcText:keypad_trace_button"
+		(property "Footprint" ""
 			(at 132.08 71.12 0)
 			(effects
@@
 			)
 		)
-		(property "Footprint" "CalcText:keypad_trace_button"
+		(property "Footprint" ""
 			(at 132.08 121.92 0)
 			(effects
@@
 			)
 		)
-		(property "Footprint" "CalcText:keypad_trace_button"
+		(property "Footprint" ""
 			(at 189.23 58.42 0)
 			(effects
@@
 			)
 		)
-		(property "Footprint" "CalcText:keypad_trace_button"
+		(property "Footprint" ""
 			(at 113.03 83.82 0)
 			(effects
@@
 			)
 		)
-		(property "Footprint" "CalcText:keypad_trace_button"
+		(property "Footprint" ""
 			(at 74.93 45.72 0)
 			(effects
@@
 			)
 		)
-		(property "Footprint" "CalcText:keypad_trace_button"
+		(property "Footprint" ""
 			(at 132.08 96.52 0)
 			(effects
@@
 			)
 		)
-		(property "Footprint" "CalcText:keypad_trace_button"
+		(property "Footprint" ""
 			(at 93.98 58.42 0)
 			(effects
@@
 			)
 		)
-		(property "Footprint" "CalcText:keypad_trace_button"
+		(property "Footprint" ""
 			(at 113.03 96.52 0)
 			(effects
@@
 			)
 		)
-		(property "Footprint" "CalcText:keypad_trace_button"
+		(property "Footprint" ""
 			(at 132.08 58.42 0)
 			(effects
@@
 			)
 		)
-		(property "Footprint" "CalcText:keypad_trace_button"
+		(property "Footprint" ""
 			(at 93.98 109.22 0)
 			(effects
@@
 			)
 		)
-		(property "Footprint" "CalcText:keypad_trace_button"
+		(property "Footprint" ""
 			(at 170.18 58.42 0)
 			(effects
@@
 			)
 		)
-		(property "Footprint" "CalcText:keypad_trace_button"
+		(property "Footprint" ""
 			(at 113.03 58.42 0)
 			(effects
@@
 			)
 		)
-		(property "Footprint" "CalcText:keypad_trace_button"
+		(property "Footprint" ""
 			(at 132.08 109.22 0)
 			(effects
@@
 			)
 		)
-		(property "Footprint" "CalcText:keypad_trace_button"
+		(property "Footprint" ""
 			(at 132.08 83.82 0)
 			(effects
@@
 			)
 		)
-		(property "Footprint" "CalcText:keypad_trace_button"
+		(property "Footprint" ""
 			(at 93.98 45.72 0)
 			(effects
@@
 			)
 		)
-		(property "Footprint" "CalcText:keypad_trace_button"
+		(property "Footprint" ""
 			(at 189.23 83.82 0)
 			(effects
@@
 			)
 		)
-		(property "Footprint" "CalcText:keypad_trace_button"
+		(property "Footprint" ""
 			(at 113.03 109.22 0)
 			(effects
@@
 			)
 		)
-		(property "Footprint" "CalcText:keypad_trace_button"
+		(property "Footprint" ""
 			(at 170.18 121.92 0)
 			(effects
@@
 			)
 		)
-		(property "Footprint" "CalcText:keypad_trace_button"
+		(property "Footprint" ""
 			(at 170.18 96.52 0)
 			(effects
@@
 			)
 		)
-		(property "Footprint" "CalcText:keypad_trace_button"
+		(property "Footprint" ""
 			(at 151.13 121.92 0)
 			(effects
@@
 			)
 		)
-		(property "Footprint" "CalcText:keypad_trace_button"
+		(property "Footprint" ""
 			(at 170.18 83.82 0)
 			(effects
@@
 			)
 		)
-		(property "Footprint" "CalcText:keypad_trace_button"
+		(property "Footprint" ""
 			(at 170.18 109.22 0)
 			(effects
@@
 			)
 		)
-		(property "Footprint" "CalcText:keypad_trace_button"
+		(property "Footprint" ""
 			(at 93.98 121.92 0)
 			(effects
@@
 			)
 		)
-		(property "Footprint" "CalcText:keypad_trace_button"
+		(property "Footprint" ""
 			(at 74.93 58.42 0)
 			(effects
@@
 			)
 		)
-		(property "Footprint" "CalcText:keypad_trace_button"
+		(property "Footprint" ""
 			(at 93.98 83.82 0)
 			(effects
@@
 			)
 		)
-		(property "Footprint" "CalcText:keypad_trace_button"
+		(property "Footprint" ""
 			(at 93.98 96.52 0)
 			(effects
@@
 			)
 		)
-		(property "Footprint" "CalcText:keypad_trace_button"
+		(property "Footprint" ""
 			(at 151.13 71.12 0)
 			(effects
@@
 			)
 		)
-		(property "Footprint" "CalcText:keypad_trace_button"
+		(property "Footprint" ""
 			(at 170.18 45.72 0)
 			(effects
@@
 			)
 		)
-		(property "Footprint" "CalcText:keypad_trace_button"
+		(property "Footprint" ""
 			(at 113.03 45.72 0)
 			(effects
@@
 			)
 		)
-		(property "Footprint" "CalcText:keypad_trace_button"
+		(property "Footprint" ""
 			(at 74.93 96.52 0)
 			(effects
@@
 			)
 		)
-		(property "Footprint" "CalcText:keypad_trace_button"
+		(property "Footprint" ""
 			(at 151.13 83.82 0)
 			(effects
@@
 			)
 		)
-		(property "Footprint" "CalcText:keypad_trace_button"
+		(property "Footprint" ""
 			(at 151.13 96.52 0)
 			(effects
@@
 			)
 		)
-		(property "Footprint" "CalcText:keypad_trace_button"
+		(property "Footprint" ""
 			(at 132.08 45.72 0)
 			(effects
@@
 			)
 		)
-		(property "Footprint" "CalcText:keypad_trace_button"
+		(property "Footprint" ""
 			(at 189.23 96.52 0)
 			(effects
@@
 			)
 		)
-		(property "Footprint" "CalcText:keypad_trace_button"
+		(property "Footprint" ""
 			(at 189.23 45.72 0)
 			(effects
@@
 			)
 		)
-		(property "Footprint" "CalcText:keypad_trace_button"
+		(property "Footprint" ""
 			(at 189.23 109.22 0)
 			(effects

Commit message: Refine hardware for fabrication and procurement
Parts:
- SW10, SW11, SW12, SW13, SW14, SW15, SW16, SW17, SW18, SW19, SW2, SW20, SW21, SW22, SW23, SW24, SW25, SW26, SW27, SW28, SW29, SW3, SW30, SW31, SW32, SW33, SW34, SW35, SW36, SW37, SW38, SW39, SW4, SW40, SW41, SW42, SW43, SW44, SW45, SW46, SW47, SW48, SW49, SW5, SW50, SW6, SW7, SW8, SW9: now left out of the parts list
