File: hardware/lcd-interposer/calctext-lcd-interposer.kicad_pcb (KiCad board)
At the start: 2 copper layers, 17.5 x 16.5 mm, 10 parts, among them J1 HICENDA_FPC, J2 MAINBOARD_FFC

Commit message: Finalise hardware sanity-check cleanup
Parts:
- J1: value HICENDA_FPC -> FH34SRJ-24S-0.5SH; footprint calctext-lcd-interposer:Hirose_FH34SRJ-24S-0.5SH -> CalcText_Shared:Hirose_FH34SRJ-24S-0.5SH
- J2: value MAINBOARD_FFC -> FH34SRJ-10S-0.5SH; footprint calctext-lcd-interposer:Hirose_FH34SRJ-10S-0.5SH -> CalcText_Shared:Hirose_FH34SRJ-10S-0.5SH
